File: PCB/Duino_miner.kicad_pcb (KiCad board)
At the start: 2 copper layers, 78.8 x 43.2 mm, 64 parts, among them J1 Conn_02x03_Odd_Even, Q1 BSS138PS, SW1 SW_Push, SW2 SW_Push, SW3 SW_Push, SW4 SW_Push, SW5 SW_Push, SW6 SW_Push, U1 XIAO-ESP32-C3-SMD, U2 ATmega328P-AU, U3 ATmega328P-AU, U4 ATmega328P-AU, U5 ATmega328P-AU, U6 ATmega328P-AU, U7 ATmega328P-AU, Y1 Crystal, Y2 Crystal, Y3 Crystal, Y4 Crystal, Y5 Crystal, Y6 Crystal

Commit message: 2 Chips done
Parts:
- moved C13 89.1 mm to (115.8, 79.7)
- moved C14 89.1 mm to (115.8, 82.2)
- moved C15 89.1 mm to (115.8, 84.7)
- moved C16 89.1 mm to (136.9, 79.7)
- moved C17 89.1 mm to (136.9, 82.2)
- moved C18 89.1 mm to (136.9, 84.7)
- moved C23 89.1 mm to (81.2, 79.0)
- moved C24 89.1 mm to (81.2, 81.5)
- moved C25 89.1 mm to (105.0, 76.8)
- moved C27 89.1 mm to (122.2, 82.8)
- moved C28 89.1 mm to (121.8, 78.6)
- moved C29 89.1 mm to (141.6, 79.6)
- moved C30 89.1 mm to (141.6, 82.1)
- moved C7 89.1 mm to (85.8, 81.0)
- moved C8 89.1 mm to (85.8, 83.5)
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Routing:
- net +5V: track 4.48 -> 183.3 mm
- net +3V3: track 2.87 -> 34.0 mm
- net Net-(U3-~{RESET}/PC6): track 0.00 -> 14.6 mm
- net Net-(U2-~{RESET}/PC6): track 0.00 -> 14.2 mm
- net /ISP_RESET: track 0.00 -> 13.0 mm
- net Net-(Q1B-S): track 0.00 -> 10.4 mm
- net Net-(Q1A-S): track 0.00 -> 10.2 mm
- net Net-(U3-XTAL1/PB6): track 0.00 -> 9.56 mm
- net Net-(U2-XTAL1/PB6): track 0.00 -> 9.01 mm
- net Net-(U3-XTAL2/PB7): track 0.00 -> 8.56 mm
- net Net-(U2-XTAL2/PB7): track 0.00 -> 8.29 mm
- net /SCL_5V: track 0.00 -> 4.49 mm
- net Net-(U3-AREF): track 0.00 -> 2.44 mm
- net Net-(U2-AREF): track 0.00 -> 2.38 mm
- net /SDA_5V: track 0.00 -> 2.07 mm
Other:
- board size 78.8 x 43.2 mm -> 78.8 x 70.6 mm

Commit message: PCB done, yepeee
Parts:
- added H1: MountingHole, MountingHole:MountingHole_2mm, F.Cu at (222.3, 90.0)
- added H2: MountingHole, MountingHole:MountingHole_2mm, F.Cu at (163.4, 100.7)
- moved SW3 125.4 mm to (193.8, 96.0)
- moved R3 110.5 mm to (191.1, 93.7), turned to 90 degrees
- moved SW5 107.3 mm to (213.5, 85.3), turned to 135 degrees
- moved SW4 105.7 mm to (198.8, 67.2), turned to -45 degrees
- moved U4 105.3 mm to (184.4, 95.0), turned to -90 degrees
- moved SW6 103.3 mm to (220.0, 103.9), turned to 135 degrees
- moved C9 100.3 mm to (185.0, 101.4), turned to 180 degrees
- moved C7 99.3 mm to (184.9, 88.1)
- moved C23 99.2 mm to (180.1, 87.2), turned to 45 degrees
- moved C8 97.4 mm to (181.6, 101.4)
- moved U7 96.5 mm to (217.8, 114.2), turned to -90 degrees
- moved U6 95.3 mm to (207.5, 91.3), turned to -90 degrees
- moved C24 94.8 mm to (175.5, 92.1), turned to 45 degrees
- moved Y3 93.5 mm to (173.4, 88.7), turned to 45 degrees
- moved R5 93.3 mm to (214.9, 90.0), turned to 90 degrees
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Routing:
- net +5V: track 183.3 -> 448.8 mm, vias 0 -> 1
- net /ISP_SCK: track 0.00 -> 177.7 mm, vias 0 -> 7
- net /SDA_5V: track 2.07 -> 163.9 mm, vias 0 -> 6
- net /SCL_5V: track 4.49 -> 166.2 mm, vias 0 -> 6
- net /ISP_RESET: track 13.0 -> 167.1 mm, vias 0 -> 1
- net /ISP_MOSI: track 0.00 -> 152.8 mm, vias 0 -> 8
- net /ISP_MISO: track 0.00 -> 150.7 mm, vias 0 -> 6
- net Net-(U5-~{RESET}/PC6): track 0.00 -> 23.4 mm
- net Net-(U7-~{RESET}/PC6): track 0.00 -> 22.0 mm
- net Net-(U6-~{RESET}/PC6): track 0.00 -> 17.9 mm
- net Net-(U4-~{RESET}/PC6): track 0.00 -> 12.6 mm
- net Net-(U5-XTAL2/PB7): track 0.00 -> 10.2 mm
- net Net-(U4-XTAL2/PB7): track 0.00 -> 9.70 mm
- net Net-(U6-XTAL2/PB7): track 0.00 -> 9.12 mm
- net Net-(U5-XTAL1/PB6): track 0.00 -> 9.06 mm
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- added copper zone on B.Cu, net GND
- added copper zone on F.Cu, net GND
Other:
- board size 78.8 x 70.6 mm -> 81.1 x 61.8 mm
